Commit message: Update p3dx model

File: p3dx/p3dx_description/urdf/laser/hokuyo.xacro (robot description, xacro)
@@ -31,8 +31,11 @@
       <sensor name="laser" type="ray">
         <pose>0 0 0 0 0 0</pose>
+        <visualize>true</visualize>
+        <update_rate>40</update_rate>
+        <always_on>1</always_on>
         <ray>
           <scan>
             <horizontal>
-              <!-- Hokuyo UTM-LX30 -->
+              <!-- Hokuyo UTM-30LX -->
               <resolution>1</resolution>
               <max_angle>2.356194</max_angle>              <!-- 135 Degree -->
@@ -42,5 +45,5 @@
           </scan>
           <range>
-            <min>0.10</min>
+            <min>0.1</min>
             <max>30.0</max>
             <resolution>0.01</resolution>
@@ -49,6 +52,6 @@
             <type>gaussian</type>
             <!-- Noise parameters based on published spec for Hokuyo laser achieving
-						    "+-30mm" accuracy at range < 10m. A mean of 0.0m and stddev of 0.01m will
-						    put 99.7% of samples within 0.03m of the true reading. -->
+                "+-30mm" accuracy at range < 10m. A mean of 0.0m and stddev of 0.01m will
+                put 99.7% of samples within 0.03m of the true reading. -->
             <mean>0.0</mean>
             <stddev>0.01</stddev>
@@ -57,10 +60,7 @@
         <plugin name="laser" filename="libgazebo_ros_laser.so">
           <robotNamespace></robotNamespace>
-          <topicName>/scan</topicName>
+          <topicName>scan</topicName>
           <frameName>${name}</frameName>
         </plugin>
-        <always_on>1</always_on>
-        <update_rate>40</update_rate>
-        <visualize>true</visualize>
       </sensor>
     </gazebo>

File: p3dx/p3dx_description/urdf/p3dx/pioneer3dx_body.xacro (robot description, xacro)
@@ -18,13 +18,7 @@
     <xacro:battery_block name="battery0" parent="${name}" x="-0.14" y="0.00" z="0.13" mass="2.5" />
     <!-- Wheels -->
-    <xacro:pioneer_wheel side="right" parent="${name}" xyz="0  0.15 0.09" rpy="0 0 0" radius="0.09" meshes="${meshes}"/>
-    <xacro:pioneer_wheel side="left" parent="${name}" xyz="0 -0.15 0.09" rpy="0 0 0" radius="0.09" meshes="${meshes}"/>
+    <xacro:pioneer_wheel side="right" parent="${name}" xyz="0 -0.15 0.09" rpy="0 0 0" radius="0.09" meshes="${meshes}"/>
+    <xacro:pioneer_wheel side="left" parent="${name}" xyz="0 0.15 0.09" rpy="0 0 0" radius="0.09" meshes="${meshes}"/>
     <xacro:pioneer_swivel parent="${name}" xyz="-0.185 0 0.055" rpy="0 0 0" meshes="${meshes}"/>
-    <!-- Motor plugin -->
-    <xacro:pioneer3dx_diff_drive />
-    <!-- Joints plugin -->
-    <xacro:pioneer3dx_joints_state_publisher />
-    <!-- Ground truth plugin -->
-    <xacro:pioneer3dx_ground_truth />
   </xacro:macro>
 </robot>

File: p3dx/p3dx_description/urdf/p3dx/pioneer3dx_wheel.xacro (robot description, xacro)
@@ -70,4 +70,13 @@
       <material value="Gazebo/Black"/>
     </gazebo>
+    <transmission name="${side}_wheel_trans" type="SimpleTransmission">
+      <type>transmission_interface/SimpleTransmission</type>
+      <actuator name="${side}_wheel_motor">
+        <mechanicalReduction>1</mechanicalReduction>
+      </actuator>
+      <joint name="${side}_hub_joint">
+        <hardwareInterface>hardware_interface/VelocityJointInterface</hardwareInterface>
+      </joint>
+    </transmission>
   </xacro:macro>
 </robot>

Commit message: Update Hokuyo UTM 30LX

File: p3dx/p3dx_description/urdf/laser/hokuyo.xacro (robot description, xacro)
@@ -19,5 +19,5 @@
         <origin xyz="0 0 0" rpy="0 0 0"/>
         <geometry>
-          <mesh filename="${meshes}/hokuyo.dae"/>
+          <mesh filename="${meshes}/hokuyo_utm_30lx.dae"/>
         </geometry>
       </visual>

File: p3dx/p3dx_description/urdf/p3dx/battery_block.xacro (robot description, xacro)
@@ -1,4 +1,4 @@
 <?xml version="1.0"?>
-<robot xmlns:xacro="http://ros.org/wiki/xacro">
+<robot xmlns:xacro="http://wiki.ros.org/xacro">
   <xacro:property name="M_PI" value="3.1415926535897931" />
   <xacro:macro name="battery_block" params="name parent x y z mass">

File: p3dx/p3dx_description/urdf/p3dx/inertia_tensors.xacro (robot description, xacro)
@@ -3,5 +3,5 @@
   see https://github.com/uos/uos_tools/blob/fuerte/uos_common_urdf/common.xacro and
   see http://answers.gazebosim.org/question/4372/the-inertia-matrix-explained/ -->
-<robot xmlns:xacro="http://ros.org/wiki/xacro">
+<robot xmlns:xacro="http://wiki.ros.org/xacro">
   <xacro:property name="M_PI" value="3.1415926535897931" />
   <!-- see https://secure.wikimedia.org/wikipedia/en/wiki/List_of_moment_of_inertia_tensors -->

File: p3dx/p3dx_description/urdf/p3dx/pioneer3dx.xacro (robot description, xacro)
@@ -1,4 +1,4 @@
 <?xml version="1.0"?>
-<robot xmlns:xacro="http://ros.org/wiki/xacro" name="pioneer3dx">
+<robot xmlns:xacro="http://wiki.ros.org/xacro" name="pioneer3dx">
   <!-- Import Rviz colors -->
   <xacro:include filename="$(find p3dx_description)/urdf/materials.xacro" />
@@ -7,5 +7,10 @@
   <xacro:pioneer3dx_body name="chassis" parent="base_link" meshes="package://p3dx_description/meshes/p3dx"/>
   <!-- Laser  -->
-  <xacro:include filename="$(find p3dx_description)/urdf/laser/hokuyo.xacro"/>
-  <xacro:laser name="laser" parent="chassis" xyz="0.12 0 0.26" rpy="0 0 0" meshes="package://p3dx_description/meshes/laser"/>
+  <!-- <xacro:include filename="$(find p3dx_description)/urdf/laser/hokuyo.xacro"/>
+  <xacro:laser name="laser" parent="chassis" xyz="0.12 0 0.26" rpy="0 0 0" meshes="package://p3dx_description/meshes/laser"/> -->
+  <!-- Hokuyo utm30lx -->
+  <xacro:include filename="$(find p3dx_description)/urdf/laser/hokuyo_utm30lx.urdf.xacro" />
+  <xacro:element xacro:name="sensor_hokuyo_utm30lx" prefix="sensor_hokuyo_utm30lx" parent="chassis" meshes="package://p3dx_description/meshes/laser" >
+    <origin xyz="0.12 0 0.235" rpy="0 0 0"/>
+  </xacro:element>
 </robot>

File: p3dx/p3dx_description/urdf/p3dx/pioneer3dx_body.xacro (robot description, xacro)
@@ -1,4 +1,4 @@
 <?xml version="1.0"?>
-<robot xmlns:xacro="http://ros.org/wiki/xacro">
+<robot xmlns:xacro="http://wiki.ros.org/xacro">
   <xacro:include filename="inertia_tensors.xacro"/>
   <xacro:include filename="pioneer3dx_chassis.xacro"/>

File: p3dx/p3dx_description/urdf/p3dx/pioneer3dx_chassis.xacro (robot description, xacro)
@@ -1,4 +1,4 @@
 <?xml version="1.0"?>
-<robot xmlns:xacro="http://ros.org/wiki/xacro">
+<robot xmlns:xacro="http://wiki.ros.org/xacro">
   <xacro:property name="M_PI" value="3.1415926535897931" />
   <xacro:macro name="pioneer_chassis" params="name parent xyz rpy meshes">

File: p3dx/p3dx_description/urdf/p3dx/pioneer3dx_plugins.xacro (robot description, xacro)
@@ -1,4 +1,4 @@
 <?xml version="1.0"?>
-<robot xmlns:xacro="http://ros.org/wiki/xacro">
+<robot xmlns:xacro="http://wiki.ros.org/xacro">
   <gazebo>
     <plugin name="gazebo_ros_control" filename="libgazebo_ros_control.so">

File: p3dx/p3dx_description/urdf/p3dx/pioneer3dx_sonar.xacro (robot description, xacro)
@@ -1,4 +1,4 @@
 <?xml version="1.0"?>
-<robot xmlns:xacro="http://ros.org/wiki/xacro">
+<robot xmlns:xacro="http://wiki.ros.org/xacro">
   <xacro:property name="M_PI" value="3.1415926535897931" />
   <xacro:macro name="pioneer_sonar" params="name parent xyz rpy meshes">

File: p3dx/p3dx_description/urdf/p3dx/pioneer3dx_swivel.xacro (robot description, xacro)
@@ -1,4 +1,4 @@
 <?xml version="1.0"?>
-<robot xmlns:xacro="http://ros.org/wiki/xacro">
+<robot xmlns:xacro="http://wiki.ros.org/xacro">
   <xacro:property name="M_PI" value="3.1415926535897931" />
   <xacro:macro name="pioneer_swivel" params="parent xyz rpy meshes">

File: p3dx/p3dx_description/urdf/p3dx/pioneer3dx_wheel.xacro (robot description, xacro)
@@ -1,4 +1,4 @@
 <?xml version="1.0"?>
-<robot xmlns:xacro="http://ros.org/wiki/xacro">
+<robot xmlns:xacro="http://wiki.ros.org/xacro">
   <xacro:property name="M_PI" value="3.1415926535897931" />
   <xacro:macro name="pioneer_wheel" params="side parent xyz rpy radius meshes">
